File: motor.kicad_sch (KiCad schematic)
At the start: 67 parts

Commit message: add schematic pdf
Other:
- note added: "MOTOR CONNECTORS"
- note removed: "SIGNAL CONNECTORS"
Changed lines of the file:
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@@
     (effects (font (size 1.27 1.27)) (justify left bottom))
   )
-  (text "SIGNAL CONNECTORS" (at 17.78 127 0)
+  (text "MOTOR CONNECTORS" (at 17.78 127 0)
     (effects (font (size 1.27 1.27)) (justify left bottom))
   )
